File: elec/layout/default/sk6805-ec20.kicad_pcb (KiCad board)
At the start: 2 copper layers, 225.7 x 100.8 mm, 0 parts

Commit message: initial layout
Parts:
- added C1: Multilayer Ceramic Capacitors MLCC - SMD/SMT 100nF 10V 0402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, lib:C0402, F.Cu at (164.0, 86.1)
- added U1: , lib:LED-SMD_4P-L2.0-W2.0-BR, F.Cu at (163.9, 83.9)
Routing:
- net vcc: track 0.00 -> 2.93 mm, vias 0 -> 1
- net gnd: track 0.00 -> 2.42 mm, vias 0 -> 2
Changed lines of the file:
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@@
   )
   (net 0 "")
+  (net 1 "io")
+  (net 2 "vcc")
+  (net 3 "io-1")
+  (net 4 "gnd")
+  (footprint "lib:LED-SMD_4P-L2.0-W2.0-BR" (layer "F.Cu")
+    (at 163.895 83.935)
+    (attr smd)
+    (fp_text reference "U1" (at 0 -4.65) (layer "F.SilkS") hide
+        (effects (font (size 1 1) (thickness 0.15)))
+    )
+    (fp_text value "" (at 0 4.65) (layer "F.Fab")
+        (effects (font (size 1 1) (thickness 0.15)))
+    )
+    (fp_text user "${REFERENCE}" (at 0 0) (layer "F.Fab")
+        (effects (font (size 1 1) (thickness 0.15)))
+    )
+    (fp_line (start 0.7 1.5) (end 1.5 1.5)
+      (stroke (width 0.15) (type solid)) (layer "F.SilkS"))
+    (fp_line (start 1.5 1.5) (end 1.5 0.75)
+      (stroke (width 0.15) (type solid)) (layer "F.SilkS"))
+    (fp_circle (center 0.9 0.9) (end 1 0.9)
+      (stroke (width 0.2) (type solid)) (fill none) (layer "Cmts.User"))
+    (fp_line (start -1.25 -1.25) (end -1.25 -1.25)
+      (stroke (width 3) (type solid)) (layer "F.Fab"))
+    (fp_line (start -1.25 -1.25) (end 1.25 -1.25)
+      (stroke (width 3) (type solid)) (layer "F.Fab"))
+    (fp_line (start 1.25 -1.25) (end 1.25 1.25)
+      (stroke (width 3) (type solid)) (layer "F.Fab"))
+    (fp_line (start 1.25 1.25) (end -1.25 1.25)
+      (stroke (width 3) (type solid)) (layer "F.Fab"))
+    (fp_circle (center 1 1) (end 1.03 1)
+      (stroke (width 0.06) (type solid)) (fill none) (layer "F.Fab"))
+    (pad "1" smd rect (at 0.65 0.65) (size 0.8 0.8) (layers "F.Cu" "F.Paste" "F.Mask")
+      (net 2 "vcc") (pintype "stereo"))
+    (pad "2" smd rect (at 0.65 -0.65) (size 0.8 0.8) (layers "F.Cu" "F.Paste" "F.Mask")
+      (net 1 "io") (pintype "stereo"))
+    (pad "3" smd rect (at -0.65 -0.65) (size 0.8 0.8) (layers "F.Cu" "F.Paste" "F.Mask")
+      (net 4 "gnd") (pintype "stereo"))
+    (pad "4" smd rect (at -0.65 0.65) (size 0.8 0.8) (layers "F.Cu" "F.Paste" "F.Mask")
+      (net 3 "io-1") (pintype "stereo"))
+    (model "/Users/narayanpowderly/Documents/atopile-workspace/swoop/.ato/modules/sk6805-ec20/elec/footprints/footprints.3dshapes/LED-SMD_4P-L2.0-W2.0-BR.wrl"
+      (offset (xyz 0 -0 -0))
+      (scale (xyz 1 1 1))
+      (rotate (xyz 0 0 0))
+    )
+  )
+  (footprint "lib:C0402" (layer "F.Cu")
+    (at 164.003037 86.061142 180)
+    (descr "Capacitor SMD 0402 (1005 Metric), square (rectangular) end terminal, IPC_7351 nominal, (Body size source: IPC-SM-782 page 76, https://www.pcb-3d.com/wordpress/wp-content/uploads/ipc-sm-782a_amendment_1_and_2.pdf), generated with kicad-footprint-generator")
+    (tags "capacitor")
+    (attr smd)
+    (fp_text reference "C1" (at 0 -1.16) (layer "F.SilkS") hide
+        (effects (font (size 1 1) (thickness 0.15)))
+    )
+    (fp_text value "Multilayer Ceramic Capacitors MLCC - SMD/SMT 100nF 10V 0402 RoHS" (at 0 1.16) (layer "F.Fab")
+        (effects (font (size 1 1) (thickness 0.15)))
+    )
+    (fp_text user "${REFERENCE}" (at 0 0) (layer "F.Fab")
+        (effects (font (size 0.25 0.25) (thickness 0.04)))
+    )
+    (fp_line (start -0.107836 -0.36) (end 0.107836 -0.36)
+      (stroke (width 0.12) (type solid)) (layer "F.SilkS"))
+    (fp_line (start -0.107836 0.36) (end 0.107836 0.36)
+      (stroke (width 0.12) (type solid)) (layer "F.SilkS"))
+    (fp_line (start -0.91 -0.46) (end 0.91 -0.46)
+      (stroke (width 0.05) (type solid)) (layer "F.CrtYd"))
+    (fp_line (start -0.91 0.46) (end -0.91 -0.46)
+      (stroke (width 0.05) (type solid)) (layer "F.CrtYd"))
+    (fp_line (start 0.91 -0.46) (end 0.91 0.46)
+      (stroke (width 0.05) (type solid)) (layer "F.CrtYd"))
+    (fp_line (start 0.91 0.46) (end -0.91 0.46)
+      (stroke (width 0.05) (type solid)) (layer "F.CrtYd"))
+    (fp_line (start -0.5 -0.25) (end 0.5 -0.25)
+      (stroke (width 0.1) (type solid)) (layer "F.Fab"))
+    (fp_line (start -0.5 0.25) (end -0.5 -0.25)
+      (stroke (width 0.1) (type solid)) (layer "F.Fab"))
+    (fp_line (start 0.5 -0.25) (end 0.5 0.25)
+      (stroke (width 0.1) (type solid)) (layer "F.Fab"))
+    (fp_line (start 0.5 0.25) (end -0.5 0.25)
+      (stroke (width 0.1) (type solid)) (layer "F.Fab"))
+    (pad "1" smd roundrect (at -0.48 0 180) (size 0.56 0.62) (layers "F.Cu" "F.Paste" "F.Mask") (roundrect_rratio 0.25)
+      (net 2 "vcc") (pintype "stereo"))
+    (pad "2" smd roundrect (at 0.48 0 180) (size 0.56 0.62) (layers "F.Cu" "F.Paste" "F.Mask") (roundrect_rratio 0.25)
+      (net 4 "gnd") (pintype "stereo"))
+    (model "${KICAD6_3DMODEL_DIR}/Capacitor_SMD.3dshapes/C_0402_1005Metric.wrl"
+      (offset (xyz 0 0 0))
+      (scale (xyz 1 1 1))
+      (rotate (xyz 0 0 0))
+    )
+  )
   (gr_circle (center 225.62 81.79) (end 227.32 81.79)
     (stroke (width 0.1) (type solid)) (fill none) (layer "Edge.Cuts"))
@@
       (xy 69.100734 49.778315)
     )
-    (stroke (width 0) (type solid)) (fill none) (layer "Edge.Cuts"))
+    (stroke (width 0.1) (type solid)) (fill none) (layer "Edge.Cuts"))
   (gr_arc (start 261.62 113.79) (mid 260.448427 116.618427) (end 257.62 117.79)
     (stroke (width 0.1) (type solid)) (layer "Edge.Cuts"))
@@
     (effects (font (size 2 2) (thickness 0.1)) (justify left bottom))
   )
+  (segment (start 165.159428 84.646963) (end 164.483037 84.646963) (width 0.25) (layer "F.Cu") (net 2))
+  (segment (start 164.483037 86.061142) (end 164.483037 84.646963) (width 0.25) (layer "F.Cu") (net 2))
+  (segment (start 165.68854 85.176075) (end 165.159428 84.646963) (width 0.25) (layer "F.Cu") (net 2))
+  (segment (start 164.483037 84.646963) (end 164.545 84.585) (width 0.25) (layer "F.Cu") (net 2))
+  (via (at 165.68854 85.176075) (size 0.8) (drill 0.4) (layers "F.Cu" "B.Cu") (net 2))
+  (segment (start 163.245 83.285) (end 162.044317 83.285) (width 0.25) (layer "F.Cu") (net 4))
+  (segment (start 162.044317 83.285) (end 161.985461 83.226144) (width 0.25) (layer "F.Cu") (net 4))
+  (segment (start 162.549425 86.061142) (end 162.432693 86.177874) (width 0.25) (layer "F.Cu") (net 4))
+  (segment (start 163.523037 86.061142) (end 162.549425 86.061142) (width 0.25) (layer "F.Cu") (net 4))
+  (via (at 162.432693 86.177874) (size 0.8) (drill 0.4) (layers "F.Cu" "B.Cu") (net 4))
+  (via (at 161.985461 83.226144) (size 0.8) (drill 0.4) (layers "F.Cu" "B.Cu") (net 4))
   (group "" (id 6c1ef9f7-0f34-47bb-ac1a-76df23fb396e)
     (members
