File: elec/layout/default/sk6805-ec20.kicad_pcb (KiCad board)
At the start: 2 copper layers, 225.7 x 100.8 mm, 2 parts

Commit message: Remove xmas crud
Other:
- board outline removed
- board text removed: "{{GITHASH}}"
